File: ESP32-C6-1.kicad_sch (KiCad schematic)
At the start: 38 parts, among them J1 KF301-5.0-2P, J11 Conn_02x07_Odd_Even, J12 Conn_02x02_Odd_Even, J13 Conn_02x02_Odd_Even, J2 TYPE-C-31-M-12, SW1 TS-1088-AR02016, SW2 TS-1088-AR02016, U1 USBLC6-2SC6, U2 AP63203WU-7, U3 ESP32-C6-MINI-1-N4

Commit message: README wording, schematic tweak
Clarify humidity sensor purpose (bathroom boost), add slider price,
line breaks in push/pull section.

Co-Authored-By: Claude Fable 5.1 <noreply@anthropic.com>
Other:
- note added: "?EN?"
Changed lines of the file:
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@@
 		(rev "1.0")
+	)
+	(text "?EN?"
+		(exclude_from_sim no)
+		(at 161.036 117.094 0)
+		(effects
+			(font
+				(size 1.27 1.27)
+				(color 0 0 0 1)
+			)
+		)
 	)
 	(text "5V IN / USB-Protection"
